Commit message: update cart

File: install/iiwa_description/share/iiwa_description/urdf/iiwa.urdf.xacro (robot description, xacro)
@@ -165,5 +165,5 @@
       <inertial>
         <origin xyz="0 0 0.02" rpy="0 0 0"/>
-        <mass value="${0.3 / 0.308 * 0.44}"/> <!--this is for the MFT Pneumatisch flange-->
+        <mass value="${0.3 / 0.308 * 0.44}"/>
         <inertia ixx="0.01"  ixy="0"  ixz="0" iyy="0.01" iyz="0" izz="0.01" />
       </inertial>
@@ -225,35 +225,61 @@
       <axis xyz="0 0 0"/>
   </joint>
-      <joint name="${prefix}camera_joint" type="fixed">
-        <parent link="${prefix}tool0"/>
-        <child link="${prefix}camera_link"/>
-        <origin xyz="0 0 0.02" rpy="3.14 -1.57 0"/>
-    </joint>
-    <link name="${prefix}camera_link">
-        <visual>
-          <geometry>
-            <box size="0.03 0.03 0.03"/>
-          </geometry>
-          <material name="black">
-            <color rgba="0 0 0 1"/>
-          </material>
-        </visual>
-        <collision>
-          <geometry>
-            <box size="0.03 0.03 0.03"/>
-          </geometry>
-        </collision>
-        <inertial>
-          <mass value="0.05"/>
-          <inertia ixx="0.0001" ixy="0" ixz="0" iyy="0.0001" iyz="0" izz="0.0001"/>
-        </inertial>
-    </link>
-    <joint name="${prefix}camera_optical_joint" type="fixed">
-        <parent link="${prefix}camera_link"/>
-        <child link="${prefix}camera_optical_frame"/>
-        <origin xyz="0 0 0" rpy="-1.5708 0 -1.5708"/>
-    </joint>
-    <link name="${prefix}camera_optical_frame"/>
-    <gazebo reference="${prefix}camera_link">
+  <joint name="${prefix}camera_joint" type="fixed">
+      <parent link="${prefix}tool0"/>
+      <child link="${prefix}camera_link"/>
+      <origin xyz="0.07 0.0 -0.03" rpy="3.14 -1.57 0"/>
+  </joint>
+  <link name="${prefix}camera_link">
+      <visual>
+        <geometry>
+          <box size="0.03 0.03 0.03"/>
+        </geometry>
+        <material name="black">
+          <color rgba="0 0 0 1"/>
+        </material>
+      </visual>
+      <collision>
+        <geometry>
+          <box size="0.03 0.03 0.03"/>
+        </geometry>
+      </collision>
+      <inertial>
+        <mass value="0.05"/>
+        <inertia ixx="0.0001" ixy="0" ixz="0" iyy="0.0001" iyz="0" izz="0.0001"/>
+      </inertial>
+  </link>
+  <joint name="${prefix}camera_optical_joint" type="fixed">
+      <parent link="${prefix}camera_link"/>
+      <child link="${prefix}camera_optical_frame"/>
+      <origin xyz="0 0 0" rpy="-1.5708 0 -1.5708"/>
+  </joint>
+  <link name="${prefix}camera_optical_frame"/>
+  <link name="${prefix}vacuum_gripper_link">
+    <visual>
+      <geometry>
+        <cylinder radius="0.04" length="0.02"/>
+      </geometry>
+      <material name="Black">
+        <color rgba="0.1 0.1 0.1 1"/>
+      </material>
+      <origin xyz="0 0 0.01" rpy="0 0 0"/>
+    </visual>
+    <collision>
+      <geometry>
+        <cylinder radius="0.04" length="0.02"/>
+      </geometry>
+      <origin xyz="0 0 0.01" rpy="0 0 0"/>
+    </collision>
+    <inertial>
+      <mass value="0.1"/>
+      <inertia ixx="0.0001" ixy="0" ixz="0" iyy="0.0001" iyz="0" izz="0.0001"/>
+    </inertial>
+  </link>
+  <joint name="${prefix}vacuum_gripper_joint" type="fixed">
+    <parent link="${prefix}tool0"/>
+    <child link="${prefix}vacuum_gripper_link"/>
+    <origin xyz="0 0 0" rpy="0 0 0"/>
+  </joint>
+  <gazebo reference="${prefix}camera_link">
       <sensor name="${prefix}camera" type="camera">
         <always_on>1</always_on>
@@ -279,5 +305,15 @@
         </camera>
       </sensor>
-    </gazebo>
+  </gazebo>
+  <gazebo>
+    <plugin filename="libignition-gazebo-vacuum-gripper-system.so"
+            name="ignition::gazebo::systems::VacuumGripper">
+      <self_collide>false</self_collide>
+      <link_name>${prefix}vacuum_gripper_link</link_name>
+      <suction_on_topic>/gripper/on</suction_on_topic>
+      <suction_off_topic>/gripper/off</suction_off_topic>
+      <suction_enabled>false</suction_enabled>
+    </plugin>
+  </gazebo>
   </xacro:macro>
 </robot>

File: install/ros2_fra2mo/share/ros2_fra2mo/urdf/fra2mo_base_macro.xacro (robot description, xacro)
@@ -1,9 +1,6 @@
 <?xml version="1.0"?>
-<robot  xmlns:xacro="http://www.ros.org/wiki/xacro">
+<robot xmlns:xacro="http://www.ros.org/wiki/xacro">
   <xacro:include filename="$(find ros2_fra2mo)/urdf/utility_macro.xacro" />
-  <!-- WHOLE BASE MACRO-->
-  <xacro:macro name="fra2mo_base" > <!--fb : front, back ; lr: left, right -->
-    <!-- Base properties -->
-    <xacro:property name="base_height" value="0.180" />
+  <xacro:macro name="fra2mo_base" > <xacro:property name="base_height" value="0.180" />
     <xacro:property name="base_radius" value="0.11" />
     <xacro:property name="base_mass" value="5" />
@@ -11,9 +8,7 @@
     <xacro:property name="wheel_radius" value="0.035" />
     <xacro:property name="wheel_axle" value="0.13" />
-    <!-- Actual body/chassis of the robot -->
     <link name="base_footprint">
     </link>
     <link name="base_link">
-      <!-- Inertial properties -->
       <inertial>
         <origin xyz="0 0 0" />
@@ -21,5 +16,4 @@
         <xacro:cylinder_inertia m="${base_mass}" r="${base_radius}" h="${base_height}" />
       </inertial>
-      <!-- Visual representation -->
       <visual>
         <geometry>
@@ -29,5 +23,4 @@
         <origin xyz="0 0 0" rpy="0 0 0" />
       </visual>
-      <!-- Collision properties -->
       <collision>
         <geometry>
@@ -43,5 +36,68 @@
       </collision>
     </link>
-    <!-- Left Wheel -->
+    <link name="cart_link">
+      <visual>
+        <geometry>
+          <box size="0.30 0.20 0.05"/>
+        </geometry>
+        <material name="Grey">
+          <color rgba="0.6 0.6 0.6 1"/>
+        </material>
+        <origin xyz="0 0 0" rpy="0 0 0"/>
+      </visual>
+      <visual> <origin xyz="0.16 0 0" rpy="0 0 0"/>
+        <geometry>
+          <box size="0.25 0.03 0.03"/>
+        </geometry>
+        <material name="DarkGrey">
+           <color rgba="0.3 0.3 0.3 1"/>
+        </material>
+      </visual>
+      <collision>
+        <geometry>
+          <box size="0.30 0.20 0.05"/>
+        </geometry>
+        <origin xyz="0 0 0" rpy="0 0 0"/>
+      </collision>
+      <inertial>
+        <mass value="2.0"/>
+        <inertia ixx="0.02" ixy="0" ixz="0"
+                 iyy="0.02" iyz="0"
+                 izz="0.02"/>
+      </inertial>
+    </link>
+    <joint name="cart_joint" type="fixed">
+      <parent link="base_link"/>
+      <child link="cart_link"/>
+      <origin xyz="-0.29 0 -0.02" rpy="0 0 0"/>
+    </joint>
+    <xacro:cart_wheel name="cart_wheel_rl" parent="cart_link" x="-0.05" y="0.08"  z="-0.025"/>
+    <xacro:cart_wheel name="cart_wheel_rr" parent="cart_link" x="-0.05" y="-0.08" z="-0.025"/>
+    <link name="package_link">
+      <visual>
+        <geometry>
+          <box size="0.12 0.12 0.08"/>
+        </geometry>
+        <material name="Brown">
+          <color rgba="0.6 0.4 0.2 1"/>
+        </material>
+      </visual>
+      <collision>
+        <geometry>
+          <box size="0.12 0.12 0.08"/>
+        </geometry>
+      </collision>
+      <inertial>
+        <mass value="0.25"/>
+        <inertia ixx="0.005" ixy="0" ixz="0"
+                 iyy="0.005" iyz="0"
+                 izz="0.005"/>
+      </inertial>
+    </link>
+    <joint name="package_joint" type="fixed">
+      <parent link="cart_link"/>
+      <child link="package_link"/>
+      <origin xyz="0 0 0.065" rpy="0 0 0"/>
+    </joint>
     <link name="left_wheel_link">
       <visual>
@@ -64,5 +120,4 @@
       </inertial>
     </link>
-    <!-- Right Wheel -->
     <link name="right_wheel_link">
       <visual>
@@ -85,9 +140,7 @@
       </inertial>
     </link>
-    <!-- Additional Links -->
     <link name="d435_link">
     </link>
     <link name="lidar_link" />
-    <!-- Joints -->
     <joint name="base_footprint_joint" type="fixed">
       <parent link="base_footprint" />
@@ -121,15 +174,4 @@
       <origin xyz="0.0 0.0 0.125" rpy="0 0 0" />
     </joint>
-    <!-- Gazebo Material Assignments
-    <gazebo reference="base_link">
-      <material>Gazebo/Blue</material>
-    </gazebo>
-    <gazebo reference="left_wheel_link">
-      <material>Gazebo/Black</material>
-    </gazebo>
-    <gazebo reference="right_wheel_link">
-      <material>Gazebo/Black</material>
-    </gazebo>-->
-    <!-- Transmissions -->
     <transmission name="left_wheel_joint_trans">
       <type>transmission_interface/SimpleTransmission</type>
@@ -148,5 +190,4 @@
       </actuator>
     </transmission>
-    <!-- Plugin for differential drive control in Gazebo-->
     <gazebo>
       <plugin name="ignition::gazebo::systems::DiffDrive" filename="libignition-gazebo-diff-drive-system.so">
@@ -155,50 +196,76 @@
         <wheel_separation>${wheel_axle}</wheel_separation>
         <wheel_radius>${wheel_radius}</wheel_radius>
-        <!--<frame_id>base_footprint</frame_id> TO LOOK
-        <ignition_frame_id>base_footprint</ignition_frame_id>-->
         <odom_publish_frequency>50</odom_publish_frequency>
         <topic>/cmd_vel</topic>
       </plugin>
     </gazebo>
-    <!--aruco tag-->
     <joint name="aruco_joint" type="fixed">
-    <parent link="base_link"/> <child link="aruco_link"/>
-    <origin xyz="0.10 0 0.13" rpy="0 0 0"/>
-  </joint>
-  <link name="aruco_link">
-    <visual>
-      <geometry>
-        <box size="0.08 0.08 0.001"/>
-      </geometry>
-      <material name="white">
-        <color rgba="1 1 1 1"/>
-      </material>
-    </visual>
-    <collision>
-      <geometry>
-        <box size="0.08 0.08 0.001"/>
-      </geometry>
-    </collision>
-    <inertial>
-      <mass value="0.01"/>
-      <inertia ixx="0.0001" ixy="0" ixz="0" iyy="0.0001" iyz="0" izz="0.0001"/>
-    </inertial>
-  </link>
-  <gazebo reference="aruco_link">
-    <visual>
-      <material>
-        <ambient>1 1 1 1</ambient>
-        <diffuse>1 1 1 1</diffuse>
-        <specular>0 0 0 1</specular>
-        <pbr>
-          <metal>
-            <albedo_map>/home/user/ros2_ws/src/arucotag/arucotag.png</albedo_map>
-            <roughness>0.5</roughness>
-          <metalness>0.0</metalness>
-          </metal>
-        </pbr>
-      </material>
-    </visual>
-  </gazebo>
+      <parent link="package_link"/> <child link="aruco_link"/>
+      <origin xyz="0 0 0.041" rpy="0 0 0"/>
+    </joint>
+    <link name="aruco_link">
+      <visual>
+        <geometry>
+          <box size="0.08 0.08 0.001"/>
+        </geometry>
+        <material name="white">
+          <color rgba="1 1 1 1"/>
+        </material>
+      </visual>
+      <inertial>
+        <mass value="0.01"/>
+        <inertia ixx="0.0001" ixy="0" ixz="0" iyy="0.0001" iyz="0" izz="0.0001"/>
+      </inertial>
+    </link>
+    <gazebo reference="aruco_link">
+      <visual>
+        <material>
+          <ambient>1 1 1 1</ambient>
+          <diffuse>1 1 1 1</diffuse>
+          <specular>0 0 0 1</specular>
+          <pbr>
+            <metal>
+              <albedo_map>/home/user/ros2_ws/src/arucotag/arucotag.png</albedo_map>
+              <roughness>0.5</roughness>
+            <metalness>0.0</metalness>
+            </metal>
+          </pbr>
+        </material>
+      </visual>
+    </gazebo>
+  </xacro:macro>
+  <xacro:macro name="cart_wheel" params="name parent x y z">
+    <link name="${name}">
+      <visual>
+        <geometry>
+          <cylinder radius="0.03" length="0.02"/>
+        </geometry>
+        <material name="Black">
+          <color rgba="0.1 0.1 0.1 1"/>
+        </material>
+        <origin rpy="1.5708 0 0"/>
+      </visual>
+      <collision>
+        <geometry>
+          <cylinder radius="0.03" length="0.02"/>
+        </geometry>
+        <origin rpy="1.5708 0 0"/>
+      </collision>
+      <inertial>
+        <mass value="0.1"/>
+        <inertia ixx="0.0001" ixy="0" ixz="0" iyy="0.0001" iyz="0" izz="0.0001"/>
+      </inertial>
+    </link>
+    <joint name="${name}_joint" type="fixed">
+      <parent link="${parent}"/>
+      <child link="${name}"/>
+      <origin xyz="${x} ${y} ${z}" rpy="0 0 0"/>
+    </joint>
+    <gazebo reference="${name}">
+      <mu1>0.0</mu1>
+      <mu2>0.0</mu2>
+      <kp>1000000.0</kp>
+      <kd>1.0</kd>
+    </gazebo>
   </xacro:macro>
 </robot>
