Commit message: detach update

File: install/iiwa_description/share/iiwa_description/gazebo/iiwa.gazebo.xacro (robot description, xacro)
@@ -4,5 +4,5 @@
     <!-- ros_control plugin -->
   <gazebo>
-  <plugin filename="ign_ros2_control-system" name="ign_ros2_control::IgnitionROS2ControlPlugin">
+  <plugin filename="gz_ros2_control-system" name="gz_ros2_control::GazeboSimROS2ControlPlugin">
     <ros>
       <namespace>/iiwa</namespace> </ros>
@@ -15,4 +15,15 @@
       <material>Gazebo/Gray</material>
     </gazebo>
+     <gazebo>
+      <plugin filename="libignition-gazebo-detachable-joint-system.so"
+              name="ignition::gazebo::systems::DetachableJoint">
+        <parent_link>${prefix}vacuum_gripper_link</parent_link>
+        <child_model>package</child_model>
+        <child_link>package_link</child_link>
+        <output_topic>/gripper/state</output_topic>
+        <detach_topic>/gripper/detach</detach_topic>
+        <attach_topic>/gripper/attach</attach_topic>
+      </plugin>
+    </gazebo>
   </xacro:macro>
 </robot>

File: install/iiwa_description/share/iiwa_description/ros2_control/iiwa.r2c_hardware.xacro (robot description, xacro)
@@ -6,5 +6,5 @@
             <xacro:if value="$(arg use_sim)">
                 <hardware>
-                    <plugin>ign_ros2_control/IgnitionSystem</plugin>
+                    <plugin>gz_ros2_control/GazeboSimSystem</plugin>
                 </hardware>
             </xacro:if>
@@ -12,5 +12,5 @@
                 <hardware>
                 <xacro:if value="${use_fake_hardware}">
-                    <plugin>mock_components/GenericSystem</plugin>
+                    <plugin>fake_components/GenericSystem</plugin>
                     <param name="calculate_dynamics">true</param>
                 </xacro:if>

File: install/iiwa_description/share/iiwa_description/urdf/iiwa.urdf.xacro (robot description, xacro)
@@ -265,5 +265,5 @@
       <origin xyz="0 0 0.01" rpy="0 0 0"/>
     </visual>
-    <collision>
+    <collision name="${prefix}vacuum_gripper_collision">
       <geometry>
         <cylinder radius="0.04" length="0.02"/>
@@ -306,14 +306,31 @@
       </sensor>
   </gazebo>
-  <gazebo>
-    <plugin filename="libignition-gazebo-vacuum-gripper-system.so"
-            name="ignition::gazebo::systems::VacuumGripper">
-      <self_collide>false</self_collide>
-      <link_name>${prefix}vacuum_gripper_link</link_name>
-      <suction_on_topic>/gripper/on</suction_on_topic>
-      <suction_off_topic>/gripper/off</suction_off_topic>
-      <suction_enabled>false</suction_enabled>
-    </plugin>
-  </gazebo>
+<!-- Contact sensor sul gripper_link -->
+<gazebo reference="${prefix}vacuum_gripper_link">
+  <sensor name="suction_contact" type="contact">
+    <contact>
+      <collision>${prefix}vacuum_gripper_collision</collision>
+    </contact>
+    <update_rate>30</update_rate>
+    <always_on>true</always_on>
+  </sensor>
+</gazebo>
+<gazebo reference="${prefix}vacuum_gripper_joint">
+    <preserveFixedJoint>true</preserveFixedJoint>
+    <disableFixedJointLumping>true</disableFixedJointLumping>
+</gazebo>
+<!-- DetachableJoint usa gripper_link invece di link_7
+<gazebo>
+  <plugin filename="libignition-gazebo-detachable-joint-system.so"
+          name="ignition::gazebo::systems::DetachableJoint">
+    <parent_link>${prefix}vacuum_gripper_link</parent_link>
+    <child_model>package</child_model>
+    <child_link>package_link</child_link>
+    <detach_topic>/gripper/detach</detach_topic>
+    <attach_topic>/gripper/attach</attach_topic>
+    <output_topic>/gripper/state</output_topic>
+    <joint_type>fixed</joint_type>
+  </plugin>
+</gazebo> -->
   </xacro:macro>
 </robot>

File: install/ros2_fra2mo/share/ros2_fra2mo/urdf/fra2mo_base_macro.xacro (robot description, xacro)
@@ -74,30 +74,4 @@
     <xacro:cart_wheel name="cart_wheel_rl" parent="cart_link" x="-0.05" y="0.08"  z="-0.025"/>
     <xacro:cart_wheel name="cart_wheel_rr" parent="cart_link" x="-0.05" y="-0.08" z="-0.025"/>
-    <link name="package_link">
-      <visual>
-        <geometry>
-          <box size="0.12 0.12 0.08"/>
-        </geometry>
-        <material name="Brown">
-          <color rgba="0.6 0.4 0.2 1"/>
-        </material>
-      </visual>
-      <collision>
-        <geometry>
-          <box size="0.12 0.12 0.08"/>
-        </geometry>
-      </collision>
-      <inertial>
-        <mass value="0.25"/>
-        <inertia ixx="0.005" ixy="0" ixz="0"
-                 iyy="0.005" iyz="0"
-                 izz="0.005"/>
-      </inertial>
-    </link>
-    <joint name="package_joint" type="fixed">
-      <parent link="cart_link"/>
-      <child link="package_link"/>
-      <origin xyz="0 0 0.065" rpy="0 0 0"/>
-    </joint>
     <link name="left_wheel_link">
       <visual>
@@ -200,38 +174,4 @@
       </plugin>
     </gazebo>
-    <joint name="aruco_joint" type="fixed">
-      <parent link="package_link"/> <child link="aruco_link"/>
-      <origin xyz="0 0 0.041" rpy="0 0 0"/>
-    </joint>
-    <link name="aruco_link">
-      <visual>
-        <geometry>
-          <box size="0.08 0.08 0.001"/>
-        </geometry>
-        <material name="white">
-          <color rgba="1 1 1 1"/>
-        </material>
-      </visual>
-      <inertial>
-        <mass value="0.01"/>
-        <inertia ixx="0.0001" ixy="0" ixz="0" iyy="0.0001" iyz="0" izz="0.0001"/>
-      </inertial>
-    </link>
-    <gazebo reference="aruco_link">
-      <visual>
-        <material>
-          <ambient>1 1 1 1</ambient>
-          <diffuse>1 1 1 1</diffuse>
-          <specular>0 0 0 1</specular>
-          <pbr>
-            <metal>
-              <albedo_map>/home/user/ros2_ws/src/arucotag/arucotag.png</albedo_map>
-              <roughness>0.5</roughness>
-            <metalness>0.0</metalness>
-            </metal>
-          </pbr>
-        </material>
-      </visual>
-    </gazebo>
   </xacro:macro>
   <xacro:macro name="cart_wheel" params="name parent x y z">

Commit message: update box

File: install/iiwa_description/share/iiwa_description/gazebo/iiwa.gazebo.xacro (robot description, xacro)
@@ -15,5 +15,5 @@
       <material>Gazebo/Gray</material>
     </gazebo>
-     <gazebo>
+     <!--<gazebo>
       <plugin filename="libignition-gazebo-detachable-joint-system.so"
               name="ignition::gazebo::systems::DetachableJoint">
@@ -25,5 +25,5 @@
         <attach_topic>/gripper/attach</attach_topic>
       </plugin>
-    </gazebo>
+    </gazebo> -->
   </xacro:macro>
 </robot>

File: install/ros2_fra2mo/share/ros2_fra2mo/urdf/fra2mo_base_macro.xacro (robot description, xacro)
@@ -39,10 +39,10 @@
       <visual>
         <geometry>
-          <box size="0.30 0.20 0.05"/>
+          <box size="0.3 0.20 0.05"/>
         </geometry>
         <material name="Grey">
           <color rgba="0.6 0.6 0.6 1"/>
         </material>
-        <origin xyz="0 0 0" rpy="0 0 0"/>
+        <origin xyz="-0.1 0 0" rpy="0 0 0"/>
       </visual>
       <visual> <origin xyz="0.16 0 0" rpy="0 0 0"/>
@@ -174,4 +174,44 @@
       </plugin>
     </gazebo>
+  <link name="container_link">
+    <visual>
+      <origin xyz="0 0 0.01"/>
+      <geometry><box size="0.3 0.3 0.02"/></geometry>
+      <material name="Blue_Dark"><color rgba="0 0 0.5 1"/></material>
+    </visual>
+    <visual>
+      <origin xyz="0 0.145 0.075"/>
+      <geometry><box size="0.3 0.01 0.15"/></geometry>
+      <material name="Blue_Dark"/>
+    </visual>
+    <visual>
+      <origin xyz="0 -0.145 0.075"/>
+      <geometry><box size="0.3 0.01 0.15"/></geometry>
+      <material name="Blue_Dark"/>
+    </visual>
+    <visual>
+      <origin xyz="0.145 0 0.075"/>
+      <geometry><box size="0.01 0.28 0.15"/></geometry>
+      <material name="Blue_Dark"/>
+    </visual>
+    <visual>
+      <origin xyz="-0.145 0 0.075"/>
+      <geometry><box size="0.01 0.28 0.15"/></geometry>
+      <material name="Blue_Dark"/>
+    </visual>
+    <collision>
+      <origin xyz="0 0 0.075"/>
+      <geometry><box size="0.3 0.3 0.15"/></geometry>
+    </collision>
+    <inertial>
+       <mass value="0.3"/>
+       <inertia ixx="0.008" ixy="0" ixz="0" iyy="0.008" iyz="0" izz="0.008"/>
+    </inertial>
+  </link>
+    <joint name="container_joint" type="fixed">
+      <parent link="cart_link" />
+      <child link="container_link" />
+      <origin xyz="-0.1 0.0 0.025" rpy="0 0 0" />
+    </joint>
   </xacro:macro>
   <xacro:macro name="cart_wheel" params="name parent x y z">

Commit message: waypoints update

File: install/iiwa_description/share/iiwa_description/gazebo/iiwa.gazebo.xacro (robot description, xacro)
@@ -15,5 +15,5 @@
       <material>Gazebo/Gray</material>
     </gazebo>
-     <!--<gazebo>
+     <gazebo>
       <plugin filename="libignition-gazebo-detachable-joint-system.so"
               name="ignition::gazebo::systems::DetachableJoint">
@@ -25,5 +25,5 @@
         <attach_topic>/gripper/attach</attach_topic>
       </plugin>
-    </gazebo> -->
+    </gazebo>
   </xacro:macro>
 </robot>

File: install/ros2_fra2mo/share/ros2_fra2mo/urdf/fra2mo_base_macro.xacro (robot description, xacro)
@@ -174,5 +174,5 @@
       </plugin>
     </gazebo>
-  <link name="container_link">
+ <link name="container_link">
     <visual>
       <origin xyz="0 0 0.01"/>
@@ -201,6 +201,22 @@
     </visual>
     <collision>
-      <origin xyz="0 0 0.075"/>
-      <geometry><box size="0.3 0.3 0.15"/></geometry>
+      <origin xyz="0 0 0.01"/>
+      <geometry><box size="0.3 0.3 0.02"/></geometry>
+    </collision>
+    <collision>
+      <origin xyz="0 0.145 0.075"/>
+      <geometry><box size="0.3 0.01 0.15"/></geometry>
+    </collision>
+    <collision>
+      <origin xyz="0 -0.145 0.075"/>
+      <geometry><box size="0.3 0.01 0.15"/></geometry>
+    </collision>
+    <collision>
+      <origin xyz="0.145 0 0.075"/>
+      <geometry><box size="0.01 0.28 0.15"/></geometry>
+    </collision>
+    <collision>
+      <origin xyz="-0.145 0 0.075"/>
+      <geometry><box size="0.01 0.28 0.15"/></geometry>
     </collision>
     <inertial>
